Commit message: third commit

File: urdf/ur16e_rg2_gripper1.urdf (robot description, URDF)
Before this commit: robot ur16e, 17 links, 16 joints
Joints:
- joint rg2_finger_joint1: origin xyz=0.017 0 0.108 rpy=0 -1.5707963267948966 -1.5707963267948966 -> xyz=0.105 0.017 0 rpy=0 0 0
- joint rg2_finger_joint2: origin xyz=-0.017 0 0.108 rpy=0 -1.5707963267948966 -1.5707963267948966 -> xyz=0.105 -0.017 0 rpy=0 0 0
- joint rg2_grip_vis_joint: origin xyz=0 0 0.208 rpy=0 0 0 -> xyz=0.2 0 0 rpy=-1.5707963267948966 -3.141592653589793 -1.5707963267948966
- joint rg2_leftfinger_tip_joint: origin xyz=0.095-0.0145 0.0  rpy=0 0 0 -> xyz=0.095 -0.0145 0.0 rpy=0 0 0
- joint ur5_hand_joint: parent tool0 -> flange
